File: AES42HAT.kicad_pcb (KiCad board)
At the start: 2 copper layers, 65 x 55.8 mm, 228 parts, among them J1 Raspberry_Pi_2_3, J2 Conn_02x13_Odd_Even, J8 Conn_01x03_Male, J93 Ref, J94 WCK In, J98 WCK Out, T1 74930030, T2 74930030, T3 74930030, T4 74930030, T5 74930030, T6 74930030, T7 74930030, T8 74930030, U1 LPC865M201JHI48, U10 SRC4392xPFB, U2 CS2000-CP, U20 SRC4392xPFB, U3 AT24CS32-STUM, U30 SRC4392xPFB, U4 PAM2306AYPKE, U40 SRC4392xPFB, U5 SN74LVC1T45DRL, U50 74HCT4053, U51 TLV61046ADB, U52 MIC4417, U53 TLV9052S, U6 SN74LV1T125DCK, U60 74HCT4053, U61 TLV61046ADB, U62 MIC4417, U63 TLV9052S, U70 74HCT4053, U71 TLV61046ADB, U72 MIC4417, U73 TLV9052S, U80 74HCT4053, U81 TLV61046ADB, U82 MIC4417, U83 TLV9052S, Y1 10 MHz

Commit message: Describe pin functions, and change controller pin assignments for better timer usage.
Connections:
- U1 pad 1: /~{CSC} -> /UBTD
- U1 pad 14: /UCKC -> /~{CSD}
- U1 pad 16: /UCKD -> /~{CSC}
- U1 pad 17: /BLS -> /UBTA
- U1 pad 18: /MISO -> /UBTB
- U1 pad 21: /UBTC -> /UCKD
- U1 pad 23: /UBTD -> /UCKC
- U1 pad 27: /INTC -> /~{INTC}
- U1 pad 28: /INTD -> /~{INTD}
- U1 pad 3: /~{CSD} -> /UBTC
- U1 pad 42: /BCLK -> /BCK
- U1 pad 43: /UCKB -> /UCKA
- U1 pad 44: /UCKA -> /UCKB
- U1 pad 45: /UBTB -> /~{INTB}
- U1 pad 46: /UBTA -> /~{INTA}
- U1 pad 47: /~{INTB} -> /MISO
- U1 pad 48: /~{INTA} -> /BLS

Commit message: Layout added.
Parts:
- C1, C2, C3, C4, C51, C52, C53, C61, C62, C63, C71, C72, C73, C81, C82, C83: footprint Capacitor_SMD:C_0603_1608Metric -> Library-IMM:C_0603
- C10, C11, C12, C13, C14, C15, C16, C20, C21, C22, C23, C24, C25, C26, C30, C31, C32, C33, C34, C35, C36, C40, C41, C42, C43, C44, C45, C46, C50, C55, C56, C59, C60, C65, C66, C69, C70, C75, C76, C79, C80, C85, C86, C89, C90, C91, C92, C93, C94, C95, C96, C97: footprint Capacitor_SMD:C_0402_1005Metric -> Library-IMM:C_0402
- D12, D22, D32, D42: footprint LED_SMD:LED_0402_1005Metric -> Library-IMM:LED_0402_red
- D53, D63, D73, D83: footprint Diode_SMD:D_0402_1005Metric -> Library-IMM:D_DFN1006-2A
- D54, D64, D74, D84: footprint LED_SMD:LED_0402_1005Metric -> Library-IMM:LED_0402_yellow
- D91: footprint LED_SMD:LED_0402_1005Metric -> Library-IMM:LED_0402_green
- L50, L60, L70, L80: footprint local:Coupled_Choke_Wuerth_74488540250 -> Library-IMM:L_WE_5838
- L51, L61, L71, L81: footprint Inductor_SMD:L_Wuerth_MAPI-2512 -> Library-IMM:L_WE-MAPI-2512
- R1, R10, R11, R12, R14, R15, R16, R17, R2, R20, R21, R22, R24, R25, R26, R3, R30, R31, R32, R34, R36, R4, R40, R41, R42, R44, R45, R46, R5, R50, R51, R52, R53, R54, R55, R56, R57, R58, R59, R60, R61, R62, R63, R64, R65, R66, R67, R68, R69, R70, R71, R72, R73, R74, R75, R76, R77, R78, R79, R8, R80, R81, R82, R83, R84, R85, R86, R87, R88, R89, R9, R90, R91, R92, R93, R94, R96, R97: footprint Resistor_SMD:R_0402_1005Metric -> Library-IMM:R_0402
- R98, R99: footprint Resistor_SMD:R_0402_1005Metric -> Library-IMM:C_0402
- U53, U63, U73, U83: footprint Package_SO:MSOP-10_3x3mm_P0.5mm -> Library-IMM:TSOP10Q30_L10_05_11
- moved C35 0.35 mm to (93.8, 109.5)
- moved C45 0.30 mm to (80.7, 109.5)
- moved C40 0.26 mm to (76.5, 138.4)
- moved C44 0.25 mm to (69.2, 111.7)
- moved C46 0.25 mm to (69.2, 109.8)
- moved C34 0.15 mm to (82.6, 111.8)
Connections:
- R12 pad 1: Net-(D12-A) -> Net-(D12-PadA)
- R22 pad 1: Net-(D22-A) -> Net-(D22-K)
- R54 pad 2: Net-(D54-A) -> Net-(D54-K)
- R74 pad 2: Net-(D74-A) -> Net-(D74-K)
- R84 pad 2: Net-(D84-A) -> Net-(D84-K)
- R91 pad 1: Net-(D91-A) -> Net-(D91-PadA)
Routing:
- net GNDD: track 0.00 -> 4.19 mm, vias 0 -> 4
- net +3.3V: track 0.00 -> 4.00 mm, vias 0 -> 3
- net Net-(U40-RX4-): track 0.00 -> 1.78 mm
- added copper zone on In1.Cu, net GNDD
Other:
- copper layers 2 -> 6
- rule pad_to_mask_clearance: 0 -> 0.05

Commit message: PCB update.
Parts:
- C1, C2, C3, C4, C51, C52, C53, C61, C62, C63, C71, C72, C73, C81, C82, C83: footprint Library-IMM:C_0603 -> Capacitor_SMD:C_0603_1608Metric
- C10, C11, C12, C13, C14, C15, C16, C20, C21, C22, C23, C24, C25, C26, C30, C31, C32, C33, C34, C35, C36, C40, C41, C42, C43, C44, C45, C46, C50, C55, C56, C59, C60, C65, C66, C69, C70, C75, C76, C79, C80, C85, C86, C89, C90, C91, C92, C93, C94, C95, C96, C97: footprint Library-IMM:C_0402 -> Capacitor_SMD:C_0402_1005Metric
- D12, D22, D32, D42: footprint Library-IMM:LED_0402_red -> LED_SMD:LED_0402_1005Metric
- D53, D63, D73, D83: footprint Library-IMM:D_DFN1006-2A -> Diode_SMD:D_0402_1005Metric
- D54, D64, D74, D84: footprint Library-IMM:LED_0402_yellow -> LED_SMD:LED_0402_1005Metric
- D91: footprint Library-IMM:LED_0402_green -> LED_SMD:LED_0402_1005Metric
- L50, L60, L70, L80: footprint Library-IMM:L_WE_5838 -> AES42HAT:Coupled_Choke_Wuerth_74488540250
- L51, L61, L71, L81: footprint Library-IMM:L_WE-MAPI-2512 -> Inductor_SMD:L_Wuerth_MAPI-2512
- R1, R10, R11, R12, R14, R15, R16, R17, R2, R20, R21, R22, R24, R25, R26, R3, R30, R31, R32, R34, R36, R4, R40, R41, R42, R44, R45, R46, R5, R50, R51, R52, R53, R54, R55, R56, R57, R58, R59, R60, R61, R62, R63, R64, R65, R66, R67, R68, R69, R70, R71, R72, R73, R74, R75, R76, R77, R78, R79, R8, R80, R81, R82, R83, R84, R85, R86, R87, R88, R89, R9, R90, R91, R92, R93, R94, R96, R97: footprint Library-IMM:R_0402 -> Resistor_SMD:R_0402_1005Metric
- R98, R99: footprint Library-IMM:C_0402 -> Resistor_SMD:R_0402_1005Metric
- T1, T2, T3, T4, T5, T6, T7, T8: footprint local:Transformer_Wuerth_74930030 -> AES42HAT:Transformer_Wuerth_74930030
- U53, U63, U73, U83: footprint Library-IMM:TSOP10Q30_L10_05_11 -> Package_SO:MSOP-10_3x3mm_P0.5mm
- moved R46 36.3 mm to (70.2, 136.8), turned to 90 degrees
- moved R16 25.7 mm to (120.3, 136.6), turned to 90 degrees
- moved R36 23.9 mm to (83.5, 136.7), turned to 90 degrees
- moved R64 17.3 mm to (105.8, 133.5), turned to -90 degrees
- moved R74 16.3 mm to (82.4, 133.5)
- moved R26 16.3 mm to (107.0, 136.7), turned to 90 degrees
- moved D84 13.9 mm to (69.1, 135.4)
- moved R72 12.3 mm to (89.4, 129.0), turned to 90 degrees
- moved D64 12.2 mm to (105.8, 135.5), turned to 90 degrees
- moved D74 12.2 mm to (82.4, 135.4), turned to 90 degrees
- moved R61 12.0 mm to (113.8, 128.5), turned to -90 degrees
- moved R84 11.9 mm to (69.1, 133.5), turned to -90 degrees
- moved C45 11.7 mm to (69.2, 111.9)
- moved C44 11.6 mm to (80.7, 109.5)
- moved R81 11.1 mm to (77.2, 129.0)
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Connections:
- J1 pad 14: GNDD -> (no net)
- J1 pad 4: +5V -> /RCLK
- J1 pad 5: /SCL -> +3.3V
- J1 pad 6: GNDD -> (no net)
- R12 pad 1: Net-(D12-PadA) -> Net-(D12-A)
- R22 pad 1: Net-(D22-K) -> Net-(D22-A)
- R54 pad 2: Net-(D54-K) -> Net-(D54-A)
- R74 pad 2: Net-(D74-K) -> Net-(D74-A)
- R84 pad 2: Net-(D84-K) -> Net-(D84-A)
- R91 pad 1: Net-(D91-PadA) -> Net-(D91-A)
Routing:
- net /RCLK: track 0.00 -> 145.4 mm, vias 0 -> 6
- net +3.3V: track 4.00 -> 139.4 mm, vias 3 -> 26
- net /MCLK: track 0.00 -> 118.0 mm, vias 0 -> 5
- net /ACLK: track 0.00 -> 109.4 mm, vias 0 -> 6
- net /BCK: track 0.00 -> 102.3 mm, vias 0 -> 3
- net /WCLK: track 0.00 -> 100.2 mm, vias 0 -> 6
- net +1V8: track 0.00 -> 93.8 mm, vias 0 -> 8
- net /MOSI: track 0.00 -> 91.4 mm, vias 0 -> 5
- net /SCL: track 0.00 -> 87.8 mm, vias 0 -> 2
- net /SDA: track 0.00 -> 86.9 mm, vias 0 -> 2
- net /SCLK: track 0.00 -> 84.7 mm, vias 0 -> 5
- net /~{RESET}: track 0.00 -> 83.0 mm, vias 0 -> 5
- net /MISO: track 0.00 -> 79.3 mm, vias 0 -> 5
- net GNDD: track 4.19 -> 80.3 mm, vias 4 -> 106
- net /MID: track 0.00 -> 75.5 mm, vias 0 -> 7
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- added copper zone on F.Cu, net +1V8
- added copper zone on F.Cu, net +3.3V
- added copper zone on In2.Cu, net +3.3V
- added copper zone on In2.Cu, net +3.3VP
- added copper zone on F.Cu, net +5V
- added copper zone on In2.Cu, net +5V
- added copper zone on F.Cu, net GNDD
- added copper zone on In4.Cu, net GNDD
- added copper zone on F.Cu, net Net-(U51-SW)
- added copper zone on F.Cu, net Net-(U61-SW)
- added copper zone on F.Cu, net Net-(U71-SW)
- added copper zone on F.Cu, net Net-(U81-SW)
Other:
- rule solder_mask_min_width: 0.1 -> 0.05

Commit message: Layout update.
Parts:
- added C58: 100n, Capacitor_SMD:C_0402_1005Metric, F.Cu at (129.1, 116.3)
- added C68: 100n, Capacitor_SMD:C_0402_1005Metric, F.Cu at (115.8, 116.3)
- added C78: 100n, Capacitor_SMD:C_0402_1005Metric, F.Cu at (92.5, 116.3)
- added C88: 100n, Capacitor_SMD:C_0402_1005Metric, F.Cu at (79.2, 116.2)
Routing:
- net +5V: track 23.6 -> 26.3 mm
- net /~{CSD}: track 23.1 -> 23.6 mm
- net GNDD: vias 106 -> 110
Other:
- board text added: "AES42HAT"
- board text added: "s13n"
