File: AES42HAT.kicad_sch (KiCad schematic)
At the start: 228 parts, among them J1 Raspberry_Pi_2_3, J2 Conn_02x13_Odd_Even, J8 Conn_01x03_Male, J93 Ref, J94 WCK In, J98 WCK Out, T1 74930030, T2 74930030, T3 74930030, T4 74930030, T5 74930030, T6 74930030, T7 74930030, T8 74930030, U1 LPC865M201JHI48, U10 SRC4392xPFB, U2 CS2000-CP, U20 SRC4392xPFB, U3 AT24CS32-STUM, U30 SRC4392xPFB, U4 PAM2306AYPKE, U40 SRC4392xPFB, U5 SN74LVC1T45DRL, U50 74HCT4053, U51 TLV61046ADB, U52 MIC4417, U53 TLV9052S, U6 SN74LV1T125DCK, U60 74HCT4053, U61 TLV61046ADB, U62 MIC4417, U63 TLV9052S, U70 74HCT4053, U71 TLV61046ADB, U72 MIC4417, U73 TLV9052S, U80 74HCT4053, U81 TLV61046ADB, U82 MIC4417, U83 TLV9052S, Y1 10 MHz

Commit message: Describe pin functions, and change controller pin assignments for better timer usage.
Connections:
- net BCLK is gone; now on net BCK: U1.42 (PIO0_30)
- net INTC is gone; now on net ~{INTC}: U1.27 (PIO1_5)
- net INTD is gone; now on net ~{INTD}: U1.28 (PIO1_6)
- net BLS: now also U1.48 (PIO0_17); no longer U1.17 (PIO0_27)
- net MISO: now also U1.47 (PIO0_18); no longer U1.18 (PIO0_26)
- net UBTA: now also U1.17 (PIO0_27); no longer U1.46 (PIO0_19)
- net UBTB: now also U1.18 (PIO0_26); no longer U1.45 (PIO0_20)
- net UBTC: now also U1.3 (PIO1_9); no longer U1.21 (PIO1_3)
- net UBTD: now also U1.1 (PIO1_8); no longer U1.23 (PIO1_4)
- net UCKA: now also U1.43 (PIO0_22); no longer U1.44 (PIO0_21)
- net UCKB: now also U1.44 (PIO0_21); no longer U1.43 (PIO0_22)
- net UCKC: now also U1.23 (PIO1_4); no longer U1.14 (PIO1_1)
- net UCKD: now also U1.21 (PIO1_3); no longer U1.16 (PIO1_2)
- net ~{CSC}: now also U1.16 (PIO1_2); no longer U1.1 (PIO1_8)
- net ~{CSD}: now also U1.14 (PIO1_1); no longer U1.3 (PIO1_9)
- net ~{INTA}: now also U1.46 (PIO0_19); no longer U1.48 (PIO0_17)
- net ~{INTB}: now also U1.45 (PIO0_20); no longer U1.47 (PIO0_18)
Changed lines of the file:
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@@
 		)
 	)
-	(label "BCLK"
+	(label "BCK"
 		(at 544.83 55.88 180)
 		(fields_autoplaced yes)
@@
 	)
 	(label "UCKD"
-		(at 544.83 68.58 180)
+		(at 544.83 71.12 180)
 		(fields_autoplaced yes)
 		(effects
@@
 	)
 	(label "UBTD"
-		(at 544.83 73.66 180)
+		(at 544.83 83.82 180)
 		(fields_autoplaced yes)
 		(effects
@@
 	)
 	(label "~{CSC}"
-		(at 544.83 83.82 180)
+		(at 544.83 68.58 180)
 		(fields_autoplaced yes)
 		(effects
@@
 	)
 	(label "~{CSD}"
-		(at 544.83 86.36 180)
+		(at 544.83 66.04 180)
 		(fields_autoplaced yes)
 		(effects
@@
 	)
 	(label "UCKB"
-		(at 490.22 96.52 0)
+		(at 490.22 93.98 0)
 		(fields_autoplaced yes)
 		(effects
@@
 	)
 	(label "MISO"
-		(at 544.83 45.72 180)
-		(fields_autoplaced yes)
-		(effects
-			(font
-				(size 1.27 1.27)
-			)
-			(justify right bottom)
+		(at 490.22 86.36 0)
+		(fields_autoplaced yes)
+		(effects
+			(font
+				(size 1.27 1.27)
+			)
+			(justify left bottom)
 		)
 	)
@@
 	)
 	(label "BLS"
-		(at 544.83 48.26 180)
-		(fields_autoplaced yes)
-		(effects
-			(font
-				(size 1.27 1.27)
-			)
-			(justify right bottom)
+		(at 490.22 83.82 0)
+		(fields_autoplaced yes)
+		(effects
+			(font
+				(size 1.27 1.27)
+			)
+			(justify left bottom)
 		)
 	)
@@
 		)
 	)
-	(label "INTD"
+	(label "~{INTD}"
 		(at 544.83 78.74 180)
 		(fields_autoplaced yes)
@@
 		)
 	)
-	(label "INTC"
+	(label "~{INTC}"
 		(at 544.83 76.2 180)
 		(fields_autoplaced yes)
@@
 	)
 	(label "UCKC"
-		(at 544.83 66.04 180)
+		(at 544.83 73.66 180)
 		(fields_autoplaced yes)
 		(effects
@@
 	)
 	(label "~{INTA}"
-		(at 490.22 83.82 0)
+		(at 490.22 88.9 0)
 		(fields_autoplaced yes)
 		(effects
@@
 	)
 	(label "UBTA"
-		(at 490.22 88.9 0)
-		(fields_autoplaced yes)
-		(effects
-			(font
-				(size 1.27 1.27)
-			)
-			(justify left bottom)
+		(at 544.83 48.26 180)
+		(fields_autoplaced yes)
+		(effects
+			(font
+				(size 1.27 1.27)
+			)
+			(justify right bottom)
 		)
 	)
@@
 	)
 	(label "UCKA"
-		(at 490.22 93.98 0)
+		(at 490.22 96.52 0)
 		(fields_autoplaced yes)
 		(effects
@@
 	)
 	(label "~{INTB}"
-		(at 490.22 86.36 0)
+		(at 490.22 91.44 0)
 		(fields_autoplaced yes)
 		(effects
@@
 	)
 	(label "UBTB"
-		(at 490.22 91.44 0)
-		(fields_autoplaced yes)
-		(effects
-			(font
-				(size 1.27 1.27)
-			)
-			(justify left bottom)
+		(at 544.83 45.72 180)
+		(fields_autoplaced yes)
+		(effects
+			(font
+				(size 1.27 1.27)
+			)
+			(justify right bottom)
 		)
 	)
@@
 	)
 	(label "UBTC"
-		(at 544.83 71.12 180)
-		(fields_autoplaced yes)
-		(effects
+		(at 544.83 86.36 180)
+		(fields_autoplaced yes)
+		(effects

Commit message: Layout added.
Parts:
- C1, C2, C3, C4, C51, C52, C53, C61, C62, C63, C71, C72, C73, C81, C82, C83: footprint Capacitor_SMD:C_0603_1608Metric -> Library-IMM:C_0603
- C10, C11, C12, C13, C14, C15, C16, C20, C21, C22, C23, C24, C25, C26, C30, C31, C32, C33, C34, C35, C36, C40, C41, C42, C43, C44, C45, C46, C50, C55, C56, C59, C60, C65, C66, C69, C70, C75, C76, C79, C80, C85, C86, C89, C90, C91, C92, C93, C94, C95, C96, C97: footprint Capacitor_SMD:C_0402_1005Metric -> Library-IMM:C_0402
- D12, D22, D32, D42: footprint LED_SMD:LED_0402_1005Metric -> Library-IMM:LED_0402_red; symbol Device:LED_Small_Filled -> Library-IMM:LED_Small_Filled
- D53, D63, D73, D83: footprint Diode_SMD:D_0402_1005Metric -> Library-IMM:D_DFN1006-2A; symbol Device:D_Zener_Small -> Library-IMM:D_Zener_Small_Filled
- D54, D64, D74, D84: footprint LED_SMD:LED_0402_1005Metric -> Library-IMM:LED_0402_yellow; symbol Device:LED_Small_Filled -> Library-IMM:LED_Small_Filled
- D91: footprint LED_SMD:LED_0402_1005Metric -> Library-IMM:LED_0402_green; symbol Device:LED_Small_Filled -> Library-IMM:LED_Small_Filled
- L50, L60, L70, L80: footprint Coupled_Choke_Wuerth_74488540250 -> Library-IMM:L_WE_5838
- L51, L61, L71, L81: footprint Inductor_SMD:L_Wuerth_MAPI-2512 -> Library-IMM:L_WE-MAPI-2512
- R1, R10, R11, R12, R14, R15, R16, R17, R2, R20, R21, R22, R24, R25, R26, R3, R30, R31, R32, R34, R36, R4, R40, R41, R42, R44, R45, R46, R5, R50, R51, R52, R53, R54, R55, R56, R57, R58, R59, R60, R61, R62, R63, R64, R65, R66, R67, R68, R69, R70, R71, R72, R73, R74, R75, R76, R77, R78, R79, R8, R80, R81, R82, R83, R84, R85, R86, R87, R88, R89, R9, R90, R91, R92, R93, R94, R96, R97: footprint Resistor_SMD:R_0402_1005Metric -> Library-IMM:R_0402
- R98, R99: footprint Resistor_SMD:R_0402_1005Metric -> Library-IMM:C_0402
- U53, U63, U73, U83: footprint Package_SO:MSOP-10_3x3mm_P0.5mm -> Library-IMM:TSOP10Q30_L10_05_11
Connections:
- net GNDD: now also D12.K, D22.K, D32.K, D42.K, D54.K, D64.K, D74.K, D84.K, D91.K; no longer D12.1 (K), D22.1 (K), D32.1 (K), D42.1 (K), D54.1 (K), D64.1 (K), D74.1 (K), D84.1 (K), D91.1 (K)
- net at R42.1: now also D42.A; no longer D42.2 (A)
- net at R32.1: now also D32.A; no longer D32.2 (A)
- net at R64.1: now also D63.A; no longer D63.2 (A)
- net at R64.2: now also D64.A; no longer D64.2 (A)
- net at R54.1: now also D53.A; no longer D53.2 (A)
- net at R54.2: now also D54.A; no longer D54.2 (A)
- net at C52.1, C53.1, D52.1 (A1)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: now also D53.K; no longer D53.1 (K)
- net at R12.1: now also D12.A; no longer D12.2 (A)
- net at R74.2: now also D74.A; no longer D74.2 (A)
- net at C72.1, C73.1, D72.1 (A1)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: now also D73.K; no longer D73.1 (K)
- net at C82.1, C83.1, D82.1 (A1)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: now also D83.K; no longer D83.1 (K)
- net at C62.1, C63.1, D62.1 (A1)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: now also D63.K; no longer D63.1 (K)
- net at R22.1: now also D22.A; no longer D22.2 (A)
- net at R84.1: now also D83.A; no longer D83.2 (A)
- net at R84.2: now also D84.A; no longer D84.2 (A)
- net at R74.1: now also D73.A; no longer D73.2 (A)
- net at R91.1: now also D91.A; no longer D91.2 (A)

Commit message: PCB update.
Parts:
- C1, C2, C3, C4, C51, C52, C53, C61, C62, C63, C71, C72, C73, C81, C82, C83: footprint Library-IMM:C_0603 -> Capacitor_SMD:C_0603_1608Metric
- C10, C11, C12, C13, C14, C15, C16, C20, C21, C22, C23, C24, C25, C26, C30, C31, C32, C33, C34, C35, C36, C40, C41, C42, C43, C44, C45, C46, C50, C55, C56, C59, C60, C65, C66, C69, C70, C75, C76, C79, C80, C85, C86, C89, C90, C91, C92, C93, C94, C95, C96, C97: footprint Library-IMM:C_0402 -> Capacitor_SMD:C_0402_1005Metric
- D12, D22, D32, D42: footprint Library-IMM:LED_0402_red -> LED_SMD:LED_0402_1005Metric; symbol Library-IMM:LED_Small_Filled -> Device:LED_Small_Filled
- D53, D63, D73, D83: footprint Library-IMM:D_DFN1006-2A -> Diode_SMD:D_0402_1005Metric; symbol Library-IMM:D_Zener_Small_Filled -> Device:D_Zener_Small
- D54, D64, D74, D84: footprint Library-IMM:LED_0402_yellow -> LED_SMD:LED_0402_1005Metric; symbol Library-IMM:LED_Small_Filled -> Device:LED_Small_Filled
- D91: footprint Library-IMM:LED_0402_green -> LED_SMD:LED_0402_1005Metric; symbol Library-IMM:LED_Small_Filled -> Device:LED_Small_Filled
- J1: footprint local:Raspberry_Pi_HAT -> Library-IMM:Raspberry_Pi_HAT
- L50, L60, L70, L80: footprint Library-IMM:L_WE_5838 -> AES42HAT:Coupled_Choke_Wuerth_74488540250
- L51, L61, L71, L81: footprint Library-IMM:L_WE-MAPI-2512 -> Inductor_SMD:L_Wuerth_MAPI-2512
- R1, R10, R11, R12, R14, R15, R16, R17, R2, R20, R21, R22, R24, R25, R26, R3, R30, R31, R32, R34, R36, R4, R40, R41, R42, R44, R45, R46, R5, R50, R51, R52, R53, R54, R55, R56, R57, R58, R59, R60, R61, R62, R63, R64, R65, R66, R67, R68, R69, R70, R71, R72, R73, R74, R75, R76, R77, R78, R79, R8, R80, R81, R82, R83, R84, R85, R86, R87, R88, R89, R9, R90, R91, R92, R93, R94, R96, R97: footprint Library-IMM:R_0402 -> Resistor_SMD:R_0402_1005Metric
- R98, R99: footprint Library-IMM:C_0402 -> Resistor_SMD:R_0402_1005Metric
- T1, T2, T3, T4, T5, T6, T7, T8: footprint local:Transformer_Wuerth_74930030 -> AES42HAT:Transformer_Wuerth_74930030
- U53, U63, U73, U83: footprint Library-IMM:TSOP10Q30_L10_05_11 -> Package_SO:MSOP-10_3x3mm_P0.5mm
Connections:
- net GNDD: now also D12.1 (K), D22.1 (K), D32.1 (K), D42.1 (K), D54.1 (K), D64.1 (K), D74.1 (K), D84.1 (K), D91.1 (K); no longer D12.K, D22.K, D32.K, D42.K, D54.K, D64.K, D74.K, D84.K, D91.K
- net at R42.1: now also D42.2 (A); no longer D42.A
- net at R32.1: now also D32.2 (A); no longer D32.A
- net at R64.1: now also D63.2 (A); no longer D63.A
- net at R64.2: now also D64.2 (A); no longer D64.A
- net at R54.1: now also D53.2 (A); no longer D53.A
- net at R54.2: now also D54.2 (A); no longer D54.A
- net at C52.1, C53.1, D52.1 (A1)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: now also D53.1 (K); no longer D53.K
- net at R12.1: now also D12.2 (A); no longer D12.A
- net at R74.2: now also D74.2 (A); no longer D74.A
- net at C72.1, C73.1, D72.1 (A1)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: now also D73.1 (K); no longer D73.K
- net at C82.1, C83.1, D82.1 (A1)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: now also D83.1 (K); no longer D83.K
- net at C62.1, C63.1, D62.1 (A1)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: now also D63.1 (K); no longer D63.K
- net at R22.1: now also D22.2 (A); no longer D22.A
- net at R84.1: now also D83.2 (A); no longer D83.A
- net at R84.2: now also D84.2 (A); no longer D84.A
- net at R74.1: now also D73.2 (A); no longer D73.A
- net at R91.1: now also D91.2 (A); no longer D91.A

Commit message: Add a couple of blocking caps, and mark connectors as don't populate.
Parts:
- added C58 (x2), C78, C88: 100n, Capacitor_SMD:C_0402_1005Metric, symbol Device:C
- J1, J2, J8: now not fitted
Connections:
- net +5V: now also C58.1, C58.1, C78.1, C88.1
- net GNDD: now also C58.2, C58.2, C78.2, C88.2

Commit message: U3 als unbestückt markiert
Parts:
- U3: now not fitted
Changed lines of the file:
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@@
 		(in_bom yes)
 		(on_board yes)
-		(dnp no)
+		(dnp yes)
 		(fields_autoplaced yes)
 		(property "Reference" "U3"

Commit message: Layout update.
Parts:
- renumbered C58 to C68
Changed lines of the file:
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@@
 		(on_board yes)
 		(dnp no)
-		(property "Reference" "C58"
+		(property "Reference" "C68"
 			(at 188.468 220.218 0)
 			(effects
@@
 			(project "AES42HAT"
 				(path "/e63e39d7-6ac0-4ffd-8aa3-1841a4541b55"
-					(reference "C58")
+					(reference "C68")
 					(unit 1)
 				)
